File: hardware/board.sch (EAGLE design)
At the start: 131 parts, among them CON2 USB-FPGA-2THT, IC1 THS3062, IC2 AD80XX, U1 AD9215BRUZ, X1 BU-SMA-V

Commit message: Fully routed ADC
Other:
- note removed: "TODO: * GPIO2 * ADC * check everything * check CLK pins * check GPI0 uC pins Add notes where useful"
Changed lines of the file:
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@@
 <plain>
 <text x="167.64" y="137.16" size="1.778" layer="97" rot="R90">Input from power supply</text>
-<text x="147.32" y="83.82" size="1.6764" layer="150">TODO:
-* GPIO2
-* ADC
-* check everything
-* check CLK pins
-* check GPI0 uC pins
-Add notes where useful</text>
 <text x="30.48" y="147.32" size="1.016" layer="97" rot="R180" align="center-right">SC_IO was here in adapter version,
 but this is an MCU pin</text>

Commit message: Board updates Tweaks to LPC First attempt for faultfinder stm32f100
Parts:
- C19: value 10n -> 100n
Changed lines of the file:
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@@
 <part name="R_GND1" library="rcl" deviceset="R-EU_" device="R0805" value="0"/>
 <part name="GND7" library="supply1" deviceset="GND" device=""/>
-<part name="C19" library="rcl" deviceset="C-EU" device="C0805K" value="10n"/>
+<part name="C19" library="rcl" deviceset="C-EU" device="C0805K" value="100n"/>
 <part name="GND17" library="supply1" deviceset="GND" device=""/>
 <part name="TP_5V" library="testpad" deviceset="TP" device="B1,27" value="TPB1,27"/>
